File: hardware/multicdc/multicdc.kicad_sch (KiCad schematic)
At the start: 35 parts, among them J1 Conn_02x04_Odd_Even, J10 Conn_01x08_Pin, J2 Conn_02x04_Odd_Even, J3 Conn_02x04_Odd_Even, J4 Conn_02x04_Odd_Even, J5 Conn_02x04_Odd_Even, J6 Conn_02x04_Odd_Even, J7 Conn_01x06_Pin, J8 Conn_01x06_Pin, J9 Conn_01x06_Pin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

Commit message: Finish hardware designs
Other:
- note removed: "TODO extra pin headers for wire wrapping isolated power"
Changed lines of the file:
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@@
-		)
-	)
-	(text "TODO extra pin headers for wire wrapping isolated power"
-		(exclude_from_sim no)
-		(at 233.172 149.606 0)
-		(effects
-			(font
-				(size 1.27 1.27)
-			)
 		)
 	)
