File: hardware/multicdc/multicdc.kicad_pcb (KiCad board)
At the start: 2 copper layers, 54.6 x 49.5 mm, 35 parts, among them J1 Conn_02x04_Odd_Even, J10 Conn_01x08_Pin, J2 Conn_02x04_Odd_Even, J3 Conn_02x04_Odd_Even, J4 Conn_02x04_Odd_Even, J5 Conn_02x04_Odd_Even, J6 Conn_02x04_Odd_Even, J7 Conn_01x06_Pin, J8 Conn_01x06_Pin, J9 Conn_01x06_Pin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

Commit message: Finish hardware designs
Other:
- board text added: "+3V3"
- board text added: "+5V"
- board text added: "GND"
- board text added: "RX"
- board text added: "TX"
- board text added: "VCC"

Commit message: Add note to PCB
Other:
- board text added: "RP2040 holes are too small, should be 1.0mm. Library footprint updated."
